File: Hardware/GloTime.brd (EAGLE design)
At the start: 160 x 100 mm, 9 parts, among them U1 ATMEGA328P_TQFP

Commit message: Updated Board
Parts:
- removed C1, C5: 0.1u, LinnesLab-Passives:C0201
- removed C3: 22p, LinnesLab-Passives:C0201
- removed C4: 2.2u, LinnesLab-Passives:C0201
- added C10, C9: 22p, LinnesLab-Passives:C0603
- added C6, C7: 0.1u, LinnesLab-Passives:C0603
- added C8: 2.2u, LinnesLab-Passives:C0603
- added D1: (no value), LinnesLab-DiscreteSemi:USC
- added FTDI1: FTDI_DEVICE, LinnesLab-Connectors:FTDI_DEVICE
- added J1: AVR_SPI_PROG_3X2NS, LinnesLab-Connectors:2X3-NS
- added LED1, LED10, LED11, LED12, LED13, LED14, LED15, LED16, LED17, LED18, LED19, LED2, LED20, LED21, LED22, LED23, LED24, LED25, LED26, LED27, LED28, LED3, LED4, LED43, LED44, LED45, LED46, LED47, LED48, LED49, LED5, LED50, LED51, LED52, LED53, LED54, LED55, LED56, LED6, LED7, LED8, LED9: (no value), LinnesLab-LED:LED-0603
- added PHOTO1: PHOTOCELLPTH, LinnesLab-Sensors:PHOTOCELL
- added R2, R4, R5, R6: 10k, LinnesLab-Passives:R0603
- added U2: CD74HC4067SM96, SparkFun-IC-Logic:SSOP24
- added U3: PCF8523, LinnesLab-Clocks:SO8
- added XTAL2: 32.7680kHz, LinnesLab-Clocks:2-SMD.NOLEAD.2.0MMTO1.2MM
- C2: value 22p -> 1u; device LinnesLab-Passives:C0201 -> LinnesLab-Passives:C0603
- R1: device LinnesLab-Passives:R0201 -> LinnesLab-Passives:R0603
- moved C2 89.7 mm to (102.9, 29.3), turned to 180 degrees
- moved R1 87.1 mm to (106.7, 67.3)
Connections:
- removed net LD1: U1.2
- removed net LD16: U1.10
- removed net LD2: U1.1
- removed net LD3: U1.32
- removed net MODE: U1.9
- new net 3.3V: C2.1, R4.2, R5.2, U3.8
- new net 9V: R6.2
- new net A10/CHAN8: LED1.A, LED2.A, U2.23
- new net B10/CHAN9: LED3.A, LED4.A, U2.22
- new net C10/CHAN10: LED5.A, LED6.A, U2.21
- new net D10/CHAN11: LED7.A, LED8.A, U2.20
- new net E10/CHAN12: LED10.A, LED9.A, U2.19
- new net F10/CHAN13: LED11.A, LED11.C, LED12.A, U2.18
- new net G10/CHAN14: LED13.A, LED14.A, U2.17
- new net LD1/S2: U1.2, U2.14
- new net LD10: J1.1, U1.16
- new net LD11: J1.4, U1.15
- new net LD12: U1.14
- new net LD13: U1.13
- new net LD14: U1.12
- new net LD16/E: PHOTO1.2, R6.1, U1.10, U2.15
- new net LD2/S1: U1.1, U2.11
- new net LD3/S0: U1.32, U2.10
- new net LD9: J1.3, U1.17
- new net MODE/S3: U1.9, U2.13
- new net N$15: LED25.A, LED25.C, LED26.A
- new net N$16: LED15.A, LED16.A
- new net N$17: LED17.A, LED18.A
- new net N$18: LED19.A, LED20.A
- new net N$19: LED27.A, LED28.A
- new net N$20: LED23.A, LED24.A
- new net N$21: LED21.A, LED22.A
- new net N$29: LED53.A, LED53.C, LED54.A
- new net N$3: U3.2, XTAL2.P$1
- new net N$30: LED43.A, LED44.A
- new net N$31: LED45.A, LED46.A
- new net N$32: LED47.A, LED48.A
- new net N$33: LED55.A, LED56.A
- new net N$34: LED51.A, LED52.A
- new net N$35: LED49.A, LED50.A
- new net N$4: U3.1, XTAL2.P$2
- new net N$6: D1.+, FTDI1.VCC
- new net N$7: R2.1, U2.1
- new net SCL: R4.1, U3.6
- new net SDA: R5.1, U3.5
- new net VBATT: U3.3
- net DTR: now also C6.1, FTDI1.DTR; no longer C1.1
- net GND: now also C10.2, C7.2, C8.2, C9.2, FTDI1.CTS, FTDI1.GND, J1.6, PHOTO1.1, U3.4; no longer C3.2, C4.2, C5.2
- net N$1: now also C10.1; no longer C3.1
- net N$2: now also C9.1; no longer C2.1
- net N$5: now also C7.1, C8.1; no longer C4.1, C5.1
- net RESET: now also C6.2, J1.5, R1.1; no longer C1.2, R1.2
- net RXD: now also FTDI1.TXO
- net TXD: now also FTDI1.RXI
- net VCC: now also D1.-, J1.2, R1.2, R2.2; no longer R1.1
