File: Hardware/GloTime.sch (EAGLE design)
At the start: 9 parts, among them U1 ATMEGA328P_TQFP

Commit message: Updated Schematic
Parts:
- removed C1, C5: 0.1u, LinnesLab-Passives:CAPACITOR0201
- removed C3: 22p, LinnesLab-Passives:CAPACITOR0201
- removed C4: 2.2u, LinnesLab-Passives:CAPACITOR0201
- added C10, C9: 22p, LinnesLab-Passives:CAPACITOR0603
- added C6, C7: 0.1u, LinnesLab-Passives:CAPACITOR0603
- added C8: 2.2u, LinnesLab-Passives:CAPACITOR0603
- added D1: (no value), LinnesLab-DiscreteSemi:SCHOTTKY-USC
- added FTDI1: FTDI_DEVICE, LinnesLab-Connectors:FTDI_DEVICE
- added J1: AVR_SPI_PROG_3X2NS, LinnesLab-Connectors:AVR_SPI_PROG_3X2NS
- added LED1, LED10, LED11, LED12, LED13, LED14, LED15, LED16, LED17, LED18, LED19, LED2, LED20, LED21, LED22, LED23, LED24, LED25, LED26, LED27, LED28, LED3, LED4, LED43, LED44, LED45, LED46, LED47, LED48, LED49, LED5, LED50, LED51, LED52, LED53, LED54, LED55, LED56, LED6, LED7, LED8, LED9: (no value), LinnesLab-LED:LED0603
- added PHOTO1: PHOTOCELLPTH, LinnesLab-Sensors:PHOTOCELLPTH
- added R2, R4, R5, R6: 10k, LinnesLab-Passives:RESISTOR0603
- added U2: CD74HC4067SM96, SparkFun-IC-Logic:74HC4067SM96
- added U3: PCF8523, LinnesLab-Clocks:PCF8523
- added XTAL2: 32.7680kHz, LinnesLab-Clocks:CRYSTALECS-.327-12.5-12-C-TR
- C2: value 22p -> 1u; device LinnesLab-Passives:CAPACITOR0201 -> LinnesLab-Passives:CAPACITOR0603
- R1: device LinnesLab-Passives:RESISTOR0201 -> LinnesLab-Passives:RESISTOR0603
Connections:
- removed net LD1: U1.D4/PD4(XCK/T0)
- removed net LD16: U1.D6/PD6(AIN0)
- removed net LD2: U1.D3/PD3(INT1)
- removed net LD3: U1.D2/PD2(INT0)
- removed net MODE: U1.D5/PD5(T1)
- new net 3.3V: C2.1, R4.2, R5.2, U3.VDD
- new net 9V: R6.2
- new net A10/CHAN8: LED1.A, LED2.A, U2.CHAN8
- new net B10/CHAN9: LED3.A, LED4.A, U2.CHAN9
- new net C10/CHAN10: LED5.A, LED6.A, U2.CHAN10
- new net D10/CHAN11: LED7.A, LED8.A, U2.CHAN11
- new net E10/CHAN12: LED10.A, LED9.A, U2.CHAN12
- new net F10/CHAN13: LED11.A, LED11.C, LED12.A, U2.CHAN13
- new net G10/CHAN14: LED13.A, LED14.A, U2.CHAN14
- new net LD1/S2: U1.D4/PD4(XCK/T0), U2.S2
- new net LD10: J1.1, U1.D12/PB4(MISO)
- new net LD11: J1.4, U1.D11/PB3(MOSI/OC2)
- new net LD12: U1.D10/PB2(SS/OC1B)
- new net LD13: U1.D9/PB1(OC1A)
- new net LD14: U1.D8/PB0(ICP)
- new net LD16/E: PHOTO1.P$2, R6.1, U1.D6/PD6(AIN0), U2.EN
- new net LD2/S1: U1.D3/PD3(INT1), U2.S1
- new net LD3/S0: U1.D2/PD2(INT0), U2.S0
- new net LD9: J1.3, U1.D13/PB5(SCK)
- new net MODE/S3: U1.D5/PD5(T1), U2.S3
- new net N$15: LED25.A, LED25.C, LED26.A
- new net N$16: LED15.A, LED16.A
- new net N$17: LED17.A, LED18.A
- new net N$18: LED19.A, LED20.A
- new net N$19: LED27.A, LED28.A
- new net N$20: LED23.A, LED24.A
- new net N$21: LED21.A, LED22.A
- new net N$29: LED53.A, LED53.C, LED54.A
- new net N$3: U3.OSCO, XTAL2.1
- new net N$30: LED43.A, LED44.A
- new net N$31: LED45.A, LED46.A
- new net N$32: LED47.A, LED48.A
- new net N$33: LED55.A, LED56.A
- new net N$34: LED51.A, LED52.A
- new net N$35: LED49.A, LED50.A
- new net N$4: U3.OSCI, XTAL2.2
- new net N$6: D1.A, FTDI1.VCC
- new net N$7: R2.1, U2.COM
- new net SCL: R4.1, U3.SCL
- new net SDA: R5.1, U3.SDA
- new net VBATT: U3.VBAT
- net DTR: now also C6.1, FTDI1.DTR; no longer C1.1
- net GND: now also C10.2, C7.2, C8.2, C9.2, FTDI1.CTS, FTDI1.GND, J1.6, PHOTO1.P$1, U3.VSS; no longer C3.2, C4.2, C5.2
- net N$1: now also C10.1; no longer C3.1
- net N$2: now also C9.1; no longer C2.1
- net N$5: now also C7.1, C8.1; no longer C4.1, C5.1
- net RESET: now also C6.2, J1.5, R1.1; no longer C1.2, R1.2
- net RXD: now also FTDI1.RXI
- net TXD: now also FTDI1.TXO
- net VCC: now also D1.C, J1.2, R1.2, R2.2; no longer R1.1
Other:
- note added: "Back-up battery if desired"
- note added: "I2C Address = 0x68h"
- moved on the sheet: C2, R1, SW1, U1, XTAL_CRYSTAL-CA-310
